Commit message: restrucuted code a bit and added ground trurth estimation for the big track

File: eufsa_description/robots/imechie.urdf.xacro (robot description, xacro)
@@ -6,7 +6,7 @@
     <!-- First we import all posible elements defined in the urdf.xacro files. All these elements are defined as macro:xacros -->
     <!-- Import Robotnik CAR base elements -->
-    <xacro:include filename="$(find eufsa_description)/urdf/bases/eufsa_base.urdf.xacro" />
+    <xacro:include filename="$(find eufsa_description)/urdf/bases/imechie_base.urdf.xacro" />
     <!-- Import Robotnik CAR wheels -->
-    <xacro:include filename="$(find eufsa_description)/urdf/wheels/suspension_wheel.urdf.xacro" />
+    <!-- <xacro:include filename="$(find eufsa_description)/urdf/wheels/suspension_wheel.urdf.xacro" /> -->
     <!-- Import all available sensors -->
     <xacro:include filename="$(find eufsa_description)/sensors/all_sensors.urdf.xacro" />
@@ -33,5 +33,5 @@
     <!-- WHEELS -->
     <!-- Wheels -->
-    <xacro:front_wheel lr_prefix="left" fr_prefix="front"
+    <!-- <xacro:front_wheel lr_prefix="left" fr_prefix="front"
         lr_reflect="1" fr_reflect="1"/>
     <xacro:front_wheel lr_prefix="right" fr_prefix="front"
@@ -40,5 +40,5 @@
         lr_reflect="1" fr_reflect="-1"/>
     <xacro:rear_wheel lr_prefix="right" fr_prefix="rear"
-        lr_reflect="-1" fr_reflect="-1"/>
+        lr_reflect="-1" fr_reflect="-1"/> -->
     <!-- MAIN SENSORS -->
 <!--     LOCATIONS: (XYZ)
@@ -48,5 +48,5 @@
     STEREO CAM: -0.110 0.0 0.800 -->
     <xacro:sensor_imu parent="base_link" prefix="imu">
-        <origin xyz="0.0 0.0 0.170" rpy="0 0 0"/>
+        <origin xyz="-0.055 -0.085 0.170" rpy="0 0 0"/>
     </xacro:sensor_imu>
     <xacro:sensor_gps  parent="base_link" prefix="gps">
@@ -59,9 +59,9 @@
         <origin xyz="1.700 0.0 -0.150" rpy="0 -0.0174533 0"/>
     </xacro:VLP-16> -->
-    <xacro:VLP-16  parent="base_link" name="velodyne" topic="/velodyne_points_2" hz="10" samples="1200">
-        <origin xyz="1.700 0.0 -0.150" rpy="0 -${1.5*M_PI/180.0} 0"/>
-    </xacro:VLP-16>
+    <xacro:VLP-16R  parent="base_link" name="velodyne" topic="/velodyne_points_2" hz="8" samples="800">
+        <origin xyz="1.55 0.0 -0.242" rpy="0 ${1*M_PI/180.0} 0"/>
+    </xacro:VLP-16R>
     <xacro:zed_camera parent="base_link" prefix="zed">
-        <origin xyz="-0.110 0.0 0.8" rpy="0 0 0"/>
+        <origin xyz="1.010 0.035 0.143" rpy="0 0 0"/>
     </xacro:zed_camera>
     <!-- EXTRA SENSORS FROM THE ROBOTNIK SENSORS LIBRARY -->

File: eufsa_description/sensors/gps.urdf.xacro (robot description, xacro)
@@ -41,5 +41,5 @@
                 <bodyName>${prefix}_base_link</bodyName>
                 <!-- must be the link of the gps device, not the base_link or base_footprint -->
-                <frameId>/${prefix}_base_link</frameId>
+                <frameId>${prefix}_base_link</frameId>
                 <topicName>gps</topicName>
                 <!-- Appleton Tower coordinates -->

File: eufsa_description/sensors/imu.urdf.xacro (robot description, xacro)
@@ -35,5 +35,5 @@
 				<serviceName>${prefix}_service</serviceName>
 				<gaussianNoise>0.005</gaussianNoise>
-				<updateRate>20.0</updateRate>
+				<updateRate>1000.0</updateRate>
 			</plugin>
 		</gazebo>

File: eufsa_description/urdf/bases/eufsa_base.gazebo.xacro (robot description, xacro)
@@ -4,13 +4,27 @@
   <xacro:macro name="ros_control">
     <gazebo>
-      <plugin filename="libgazebo_ros_control.so" name="ros_control">
+      <plugin name="ros_control" filename="libgazebo_ros_control.so">
         <robotNamespace>/eufsa</robotNamespace>
         <robotParam>robot_description</robotParam>
         <!-- controlPeriod>0.003</controlPeriod -->
         <controlPeriod>0.001</controlPeriod>
-        <robotSimType>gazebo_ros_control/DefaultRobotHWSim</robotSimType>
+	    <robotSimType>gazebo_ros_control/DefaultRobotHWSim</robotSimType>
       </plugin>
     </gazebo>
-  </xacro:macro>
+	</xacro:macro>
+  <gazebo>
+    <plugin name="p3d_base_controller" filename="libgazebo_ros_p3d.so">
+        <alwaysOn>true</alwaysOn>
+        <updateRate>200.0</updateRate>
+        <bodyName>odom_ground_truth</bodyName>
+        <topicName>ground_truth/state_raw</topicName>
+        <gaussianNoise>0.00</gaussianNoise>
+        <frameName>world</frameName>
+        <!-- origin is at spawn location -->
+        <xyzOffset>43.0 -40 0</xyzOffset>
+        <rpyOffset>0 0 0</rpyOffset>
+    </plugin>
+  </gazebo>
+  <!-- No Ackermann steering plugin -->
   <gazebo reference="base_footprint">
     <material>Gazebo/Green</material>

File: eufsa_description/urdf/bases/imechie_base.urdf.xacro (robot description, xacro)
@@ -7,5 +7,5 @@
   <xacro:property name="wheel_width" value="0.175" />
   <!-- <xacro:property name="clearance" value="${tire_dia/2.0}" /> -->
-  <xacro:property name="clearance" value="0.25" />
+  <xacro:property name="clearance" value="0.397" />
   <!-- BASE FOOTPRINT -->
   <xacro:if value="${publish_bf}">
@@ -59,22 +59,4 @@
     </collision>
   </link>
-  <link name="odom_ground_truth">
-    <collision>
-      <geometry>
-        <box size="0.1 0.1 0.1"/>
-      </geometry>
-    </collision>
-    <inertial>
-      <mass value="1e-5" />
-      <origin xyz="0 0 0" rpy="0 0 0"/>
-      <inertia ixx="1e-6" ixy="0" ixz="0" iyy="1e-6" iyz="0" izz="1e-6" />
-    </inertial>
-  </link>
-  <joint name="odom_ground_truth_joint" type="fixed">
-    <axis xyz="0 0 0" />
-    <origin xyz="0 0 0" rpy="0 0 0"/>
-    <parent link="base_link"/>
-    <child link="odom_ground_truth"/>
-  </joint>
   </xacro:macro>
 </robot>

File: eufsa_description/urdf/wheels/suspension_wheel.urdf.xacro (robot description, xacro)
@@ -38,4 +38,5 @@
        (calculating this way, it should be divided by 2 if 2 motors are used)
        axle_eff_limit = 204.95 / 2 N m = ~102.5 -->
+  <!-- xacro:property name="axle_eff_limit" value="102.5"/ -->
   <xacro:property name="axle_eff_limit" value="60"/>
   <!-- max_speed = 33 Km/h = 9.17 m/s
@@ -80,4 +81,5 @@
                    ${lr_reflect * ((hex_hub_dist / 2) - axle_length)}
                    ${-wheel_travel}"/>
+                  <!-- ${(wheel_travel / 2) - shock_z_offset}"/-->
       <axis xyz="0 0 -1"/>
       <limit lower="${-wheel_travel / 2}" upper="${wheel_travel / 2}"
@@ -98,4 +100,16 @@
   <xacro:macro name="wheel" params="lr_prefix fr_prefix lr_reflect">
     <link name="${lr_prefix}_${fr_prefix}_axle_carrier">
+	  <!-- visual>
+        <origin xyz="0 0 0"/>
+        <geometry>
+          <cylinder radius="0.1" length="0.1"/>
+        </geometry>
+	  </visual>
+	  <collision>
+        <origin xyz="0 0 0"/>
+        <geometry>
+          <cylinder radius="0.1" length="0.1"/>
+        </geometry>
+	  </collision -->
       <xacro:null_inertial/>
     </link>
@@ -113,4 +127,5 @@
       <type>transmission_interface/SimpleTransmission</type>
       <joint name="${lr_prefix}_${fr_prefix}_axle">
+        <!-- hardwareInterface>hardware_interface/EffortJointInterface</hardwareInterface -->
         <hardwareInterface>hardware_interface/VelocityJointInterface</hardwareInterface>
       </joint>
@@ -148,4 +163,5 @@
     </gazebo>
   </xacro:macro>
+  <!-- xacro:macro name="rubber_wheel" params="name parent *origin reflect hq" -->
   <!-- Front wheel -->
   <xacro:macro name="front_wheel"
@@ -155,4 +171,16 @@
                  child="${lr_prefix}_steering_link"/>
     <link name="${lr_prefix}_steering_link">
+	  <!-- visual>
+		<origin xyz="0 0 0"/>
+        <geometry>
+          <cylinder radius="0.1" length="0.1"/>
+        </geometry>
+	  </visual>
+	  <collision>
+		<origin xyz="0 0 0"/>
+        <geometry>
+          <cylinder radius="0.1" length="0.1"/>
+        </geometry>
+	  </collision -->
       <xacro:null_inertial/>
     </link>
