Commit message: added ads-dv vehicle mode;

File: eufs_description/robots/ads-dv.urdf.xacro (robot description, xacro)
@@ -6,7 +6,7 @@
     <!-- First we import all posible elements defined in the urdf.xacro files. All these elements are defined as macro:xacros -->
     <!-- Import Robotnik CAR base elements -->
-    <xacro:include filename="$(find eufs_description)/urdf/bases/imechie_base.urdf.xacro" />
+    <xacro:include filename="$(find eufs_description)/urdf/bases/ads-dv_base.urdf.xacro" />
     <!-- Import Robotnik CAR wheels -->
-    <!-- <xacro:include filename="$(find eufs_description)/urdf/wheels/suspension_wheel.urdf.xacro" /> -->
+    <xacro:include filename="$(find eufs_description)/urdf/wheels/suspension_wheel.urdf.xacro" />
     <!-- Import all available sensors -->
     <xacro:include filename="$(find eufs_description)/sensors/all_sensors.urdf.xacro" />
@@ -33,5 +33,5 @@
     <!-- WHEELS -->
     <!-- Wheels -->
-    <!-- <xacro:front_wheel lr_prefix="left" fr_prefix="front"
+    <xacro:front_wheel lr_prefix="left" fr_prefix="front"
         lr_reflect="1" fr_reflect="1"/>
     <xacro:front_wheel lr_prefix="right" fr_prefix="front"
@@ -40,5 +40,5 @@
         lr_reflect="1" fr_reflect="-1"/>
     <xacro:rear_wheel lr_prefix="right" fr_prefix="rear"
-        lr_reflect="-1" fr_reflect="-1"/> -->
+        lr_reflect="-1" fr_reflect="-1"/>
     <!-- MAIN SENSORS -->
 <!--     LOCATIONS: (XYZ)
@@ -48,8 +48,8 @@
     STEREO CAM: -0.110 0.0 0.800 -->
     <xacro:sensor_imu parent="base_link" prefix="imu">
-        <origin xyz="-0.055 -0.085 0.170" rpy="0 0 0"/>
+        <origin xyz="-0.0 0.0 0.0" rpy="0 0 0"/>
     </xacro:sensor_imu>
     <xacro:sensor_gps  parent="base_link" prefix="gps">
-        <origin xyz="-0.110 0.0 0.9" rpy="0 0 0"/>
+        <origin xyz="0.0 0.0 0.4" rpy="0 0 0"/>
     </xacro:sensor_gps>
 <!--     <xacro:sensor_hokuyo_utm30lx  parent="base_link" prefix="lidar" >
@@ -60,8 +60,8 @@
     </xacro:VLP-16> -->
     <xacro:VLP-16R  parent="base_link" name="velodyne" topic="/velodyne_points_2" hz="8" samples="800">
-        <origin xyz="1.55 0.0 -0.242" rpy="0 ${1*M_PI/180.0} 0"/>
+        <origin xyz="1.58 0.0 -0.1" rpy="0 ${1*M_PI/180.0} 0"/>
     </xacro:VLP-16R>
     <xacro:zed_camera parent="base_link" prefix="zed">
-        <origin xyz="1.010 0.035 0.143" rpy="0 0 0"/>
+        <origin xyz="0.1 0.0 0.48" rpy="0 0 0"/>
     </xacro:zed_camera>
     <!-- EXTRA SENSORS FROM THE ROBOTNIK SENSORS LIBRARY -->

File: eufs_description/urdf/bases/ads-dv_base.urdf.xacro (robot description, xacro)
@@ -7,5 +7,5 @@
   <xacro:property name="wheel_width" value="0.175" />
   <!-- <xacro:property name="clearance" value="${tire_dia/2.0}" /> -->
-  <xacro:property name="clearance" value="0.397" />
+  <xacro:property name="clearance" value="0.25" />
   <!-- BASE FOOTPRINT -->
   <xacro:if value="${publish_bf}">
@@ -43,10 +43,10 @@
        <xacro:if value="${hq}">
        <geometry>
-	     <mesh filename="package://eufs_description/meshes/chassis.dae"/>
+	     <mesh filename="package://eufs_description/meshes/ads-dv.dae"/>
        </geometry>
        </xacro:if>
        <xacro:unless value="${hq}">
        <geometry>
-	     <mesh filename="package://eufs_description/meshes/chassis.dae"/>
+	     <mesh filename="package://eufs_description/meshes/ads-dv.dae"/>
        </geometry>
        </xacro:unless>
@@ -55,8 +55,26 @@
        <origin xyz="0 0 0" rpy="0 0 0 " />
        <geometry>
-         <mesh filename="package://eufs_description/meshes/chassis_collision.dae"/>
+         <mesh filename="package://eufs_description/meshes/ads-dv.dae"/>
        </geometry>
     </collision>
   </link>
+  <link name="odom_ground_truth">
+    <collision>
+      <geometry>
+        <box size="0.1 0.1 0.1"/>
+      </geometry>
+    </collision>
+    <inertial>
+      <mass value="1e-5" />
+      <origin xyz="0 0 0" rpy="0 0 0"/>
+      <inertia ixx="1e-6" ixy="0" ixz="0" iyy="1e-6" iyz="0" izz="1e-6" />
+    </inertial>
+  </link>
+  <joint name="odom_ground_truth_joint" type="fixed">
+    <axis xyz="0 0 0" />
+    <origin xyz="0 0 0" rpy="0 0 0"/>
+    <parent link="base_link"/>
+    <child link="odom_ground_truth"/>
+  </joint>
   </xacro:macro>
 </robot>

Commit message: minor sensor changes

File: eufs_description/robots/ads-dv.urdf.xacro (robot description, xacro)
@@ -59,9 +59,9 @@
         <origin xyz="1.700 0.0 -0.150" rpy="0 -0.0174533 0"/>
     </xacro:VLP-16> -->
-    <xacro:VLP-16R  parent="base_link" name="velodyne" topic="/velodyne_points_2" hz="8" samples="800">
+    <xacro:VLP-16R  parent="base_link" name="velodyne" topic="/velodyne_points" hz="10" samples="800">
         <origin xyz="1.58 0.0 -0.1" rpy="0 ${1*M_PI/180.0} 0"/>
     </xacro:VLP-16R>
     <xacro:zed_camera parent="base_link" prefix="zed">
-        <origin xyz="0.1 0.0 0.48" rpy="0 0 0"/>
+        <origin xyz="0.1 0.0 0.52" rpy="0 0 0"/>
     </xacro:zed_camera>
     <!-- EXTRA SENSORS FROM THE ROBOTNIK SENSORS LIBRARY -->

File: eufs_description/robots/eufs.urdf.xacro (robot description, xacro)
@@ -32,5 +32,4 @@
     <!-- xacro:skid_steering broadcastOdomTF="1"/ -->
     <!-- WHEELS -->
-    <!-- Wheels -->
     <xacro:front_wheel lr_prefix="left" fr_prefix="front"
         lr_reflect="1" fr_reflect="1"/>
@@ -42,9 +41,4 @@
         lr_reflect="-1" fr_reflect="-1"/>
     <!-- MAIN SENSORS -->
-<!--     LOCATIONS: (XYZ)
-    IMU: 0.0 0.0 0.170
-    GPS: -0.110 0.0 0.9
-    LIDAR: 1.700 0.0 -0.150
-    STEREO CAM: -0.110 0.0 0.800 -->
     <xacro:sensor_imu parent="base_link" prefix="imu">
         <origin xyz="0.0 0.0 0.170" rpy="0 0 0"/>
@@ -59,9 +53,9 @@
         <origin xyz="1.700 0.0 -0.150" rpy="0 -0.0174533 0"/>
     </xacro:VLP-16> -->
-    <xacro:VLP-16  parent="base_link" name="velodyne" topic="/velodyne_points_2" hz="10" samples="1200">
+    <xacro:VLP-16  parent="base_link" name="velodyne" topic="/velodyne_points" hz="10" samples="1200">
         <origin xyz="1.700 0.0 -0.150" rpy="0 -${1.5*M_PI/180.0} 0"/>
     </xacro:VLP-16>
     <xacro:zed_camera parent="base_link" prefix="zed">
-        <origin xyz="-0.110 0.0 0.8" rpy="0 0 0"/>
+        <origin xyz="-0.110 0.0 0.84" rpy="0 0 0"/>
     </xacro:zed_camera>
     <!-- EXTRA SENSORS FROM THE ROBOTNIK SENSORS LIBRARY -->
